Commit message: Made the robot blue in the description package

File: jem_355_robot_description/urdf/jem_355_robot.urdf.xacro (robot description, xacro)
@@ -28,4 +28,7 @@
         <color rgba="0.7 0.7 0.7 1" />
     </material>
+    <material name="blue">
+        <color rgba="0.5 0.5 0.9 1" />
+    </material>
     <link name="base_footprint" />
     <link name="base_link">
@@ -35,5 +38,5 @@
             </geometry>
             <origin xyz="${-base_width/2} -0.0788 0" rpy="0 0 0" />
-            <material name="gray" />
+            <material name="blue" />
         </visual>
         <collision>
